Commit message: feat(mobile_robot): 添加四轮 URDF 动力学实验和边界保护功能

File: examples/mobile_robot/assets/diff_drive_car.urdf (robot description, URDF)
Before this commit: robot genesis_diff_drive_car, 4 links, 3 joints
Links:
- removed link left_wheel
- removed link rear_caster
- removed link right_wheel
- added link front_left_wheel, mass 0.35; collision cylinder length=0.08 radius=0.13; visual cylinder length=0.08 radius=0.13
- added link front_right_wheel, mass 0.35; collision cylinder length=0.08 radius=0.13; visual cylinder length=0.08 radius=0.13
- added link rear_left_wheel, mass 0.35; collision cylinder length=0.08 radius=0.13; visual cylinder length=0.08 radius=0.13
- added link rear_right_wheel, mass 0.35; collision cylinder length=0.08 radius=0.13; visual cylinder length=0.08 radius=0.13
- link base_link: mass 4.0 -> 6.0; geometry collision box size=0.78 0.56 0.22; visual box size=0.36 0.42 0.10
Joints:
- removed joint left_wheel_joint
- removed joint rear_caster_joint
- removed joint right_wheel_joint
- added joint front_left_wheel_joint: type continuous, parent base_link, child front_left_wheel, origin xyz=0.24 0.32 0.13 rpy=0 0 0, axis 0 1 0
- added joint front_right_wheel_joint: type continuous, parent base_link, child front_right_wheel, origin xyz=0.24 -0.32 0.13 rpy=0 0 0, axis 0 1 0
- added joint rear_left_wheel_joint: type continuous, parent base_link, child rear_left_wheel, origin xyz=-0.24 0.32 0.13 rpy=0 0 0, axis 0 1 0
- added joint rear_right_wheel_joint: type continuous, parent base_link, child rear_right_wheel, origin xyz=-0.24 -0.32 0.13 rpy=0 0 0, axis 0 1 0
